File: microlidian.kicad_pcb (KiCad board)
At the start: 2 copper layers, 128.9 x 128.5 mm, 33 parts, among them J1 Eurorack power, J11 Backboard Conn 1, J12 Frontboard Conn 1, J13 Backboard Conn 2, J14 Frontboard Conn 2, J2 ST7789 TFT socket, J3 Expansion header, J4 ADS1015 digital side, J5 ADS1015 analog side, J7 TRS MIDI Out, SW1 RotaryEncoder_Switch, SW2 Back button, U1 SeeeduinoXIAO, U2 L78L05_TO92

Commit message: updated notes in readme and tracked most recent changes
Parts:
- added R5: 10K, Resistor_THT:R_Axial_DIN0207_L6.3mm_D2.5mm_P7.62mm_Horizontal, F.Cu at (85.2, 83.1)
- added R6: 10K, Resistor_THT:R_Axial_DIN0207_L6.3mm_D2.5mm_P7.62mm_Horizontal, F.Cu at (92.3, 72.9)
Routing:
- net Frontboard +3.3V: track 228.1 -> 240.5 mm
- net Encoder right Frontboard: track 84.4 -> 91.9 mm
- net Encoder left Frontboard: track 89.2 -> 93.2 mm
Changed lines of the file:
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@@
     )
   )
+  (footprint "Resistor_THT:R_Axial_DIN0207_L6.3mm_D2.5mm_P7.62mm_Horizontal" (layer "F.Cu")
+    (at 85.1662 83.1342)
+    (descr "Resistor, Axial_DIN0207 series, Axial, Horizontal, pin pitch=7.62mm, 0.25W = 1/4W, length*diameter=6.3*2.5mm^2, http://cdn-reichelt.de/documents/datenblatt/B400/1_4W%23YAG.pdf")
+    (tags "Resistor Axial_DIN0207 series Axial Horizontal pin pitch 7.62mm 0.25W = 1/4W length 6.3mm diameter 2.5mm")
+    (property "Sheetfile" "microlidian.kicad_sch")
+    (property "Sheetname" "")
+    (property "ki_description" "Resistor")
+    (property "ki_keywords" "R res resistor")
+    (attr through_hole)
+    (fp_text reference "R5" (at 3.81 -2.37) (layer "F.SilkS")
+        (effects (font (size 1 1) (thickness 0.15)))
+    )
+    (fp_text value "10K" (at 3.81 2.37) (layer "F.Fab")
+        (effects (font (size 1 1) (thickness 0.15)))
+    )
+    (fp_text user "${REFERENCE}" (at 3.81 0) (layer "F.Fab")
+        (effects (font (size 1 1) (thickness 0.15)))
+    )
+    (fp_line (start 0.54 -1.37) (end 7.08 -1.37)
+      (stroke (width 0.12) (type solid)) (layer "F.SilkS"))
+    (fp_line (start 0.54 -1.04) (end 0.54 -1.37)
+      (stroke (width 0.12) (type solid)) (layer "F.SilkS"))
+    (fp_line (start 0.54 1.04) (end 0.54 1.37)
+      (stroke (width 0.12) (type solid)) (layer "F.SilkS"))
+    (fp_line (start 0.54 1.37) (end 7.08 1.37)
+      (stroke (width 0.12) (type solid)) (layer "F.SilkS"))
+    (fp_line (start 7.08 -1.37) (end 7.08 -1.04)
+      (stroke (width 0.12) (type solid)) (layer "F.SilkS"))
+    (fp_line (start 7.08 1.37) (end 7.08 1.04)
+      (stroke (width 0.12) (type solid)) (layer "F.SilkS"))
+    (fp_line (start -1.05 -1.5) (end -1.05 1.5)
+      (stroke (width 0.05) (type solid)) (layer "F.CrtYd"))
+    (fp_line (start -1.05 1.5) (end 8.67 1.5)
+      (stroke (width 0.05) (type solid)) (layer "F.CrtYd"))
+    (fp_line (start 8.67 -1.5) (end -1.05 -1.5)
+      (stroke (width 0.05) (type solid)) (layer "F.CrtYd"))
+    (fp_line (start 8.67 1.5) (end 8.67 -1.5)
+      (stroke (width 0.05) (type solid)) (layer "F.CrtYd"))
+    (fp_line (start 0 0) (end 0.66 0)
+      (stroke (width 0.1) (type solid)) (layer "F.Fab"))
+    (fp_line (start 0.66 -1.25) (end 0.66 1.25)
+      (stroke (width 0.1) (type solid)) (layer "F.Fab"))
+    (fp_line (start 0.66 1.25) (end 6.96 1.25)
+      (stroke (width 0.1) (type solid)) (layer "F.Fab"))
+    (fp_line (start 6.96 -1.25) (end 0.66 -1.25)
+      (stroke (width 0.1) (type solid)) (layer "F.Fab"))
+    (fp_line (start 6.96 1.25) (end 6.96 -1.25)
+      (stroke (width 0.1) (type solid)) (layer "F.Fab"))
+    (fp_line (start 7.62 0) (end 6.96 0)
+      (stroke (width 0.1) (type solid)) (layer "F.Fab"))
+    (pad "1" thru_hole circle (at 0 0) (size 1.6 1.6) (drill 0.8) (layers "*.Cu" "*.Mask")
+      (net 32 "Encoder right Frontboard") (pintype "passive"))
+    (pad "2" thru_hole oval (at 7.62 0) (size 1.6 1.6) (drill 0.8) (layers "*.Cu" "*.Mask")
+      (net 51 "Frontboard +3.3V") (pintype "passive"))
+    (model "${KICAD6_3DMODEL_DIR}/Resistor_THT.3dshapes/R_Axial_DIN0207_L6.3mm_D2.5mm_P7.62mm_Horizontal.wrl"
+      (offset (xyz 0 0 0))
+      (scale (xyz 1 1 1))
+      (rotate (xyz 0 0 0))
+    )
+  )
   (footprint "Connector_PinHeader_2.54mm:PinHeader_1x08_P2.54mm_Vertical" (layer "F.Cu")
     (at 66.6498 141.2996 -90)
@@
     )
   )
+  (footprint "Resistor_THT:R_Axial_DIN0207_L6.3mm_D2.5mm_P7.62mm_Horizontal" (layer "F.Cu")
+    (at 92.3036 72.8726 180)
+    (descr "Resistor, Axial_DIN0207 series, Axial, Horizontal, pin pitch=7.62mm, 0.25W = 1/4W, length*diameter=6.3*2.5mm^2, http://cdn-reichelt.de/documents/datenblatt/B400/1_4W%23YAG.pdf")
+    (tags "Resistor Axial_DIN0207 series Axial Horizontal pin pitch 7.62mm 0.25W = 1/4W length 6.3mm diameter 2.5mm")
+    (property "Sheetfile" "microlidian.kicad_sch")
+    (property "Sheetname" "")
+    (property "ki_description" "Resistor")
+    (property "ki_keywords" "R res resistor")
+    (attr through_hole)
+    (fp_text reference "R6" (at 3.81 -2.37) (layer "F.SilkS")
+        (effects (font (size 1 1) (thickness 0.15)))
+    )
+    (fp_text value "10K" (at 3.81 2.37) (layer "F.Fab")
+        (effects (font (size 1 1) (thickness 0.15)))
+    )
+    (fp_text user "${REFERENCE}" (at 3.81 0) (layer "F.Fab")
+        (effects (font (size 1 1) (thickness 0.15)))
+    )
+    (fp_line (start 0.54 -1.37) (end 7.08 -1.37)
+      (stroke (width 0.12) (type solid)) (layer "F.SilkS"))
+    (fp_line (start 0.54 -1.04) (end 0.54 -1.37)
+      (stroke (width 0.12) (type solid)) (layer "F.SilkS"))
+    (fp_line (start 0.54 1.04) (end 0.54 1.37)
+      (stroke (width 0.12) (type solid)) (layer "F.SilkS"))
+    (fp_line (start 0.54 1.37) (end 7.08 1.37)
+      (stroke (width 0.12) (type solid)) (layer "F.SilkS"))
+    (fp_line (start 7.08 -1.37) (end 7.08 -1.04)
+      (stroke (width 0.12) (type solid)) (layer "F.SilkS"))
+    (fp_line (start 7.08 1.37) (end 7.08 1.04)
+      (stroke (width 0.12) (type solid)) (layer "F.SilkS"))
+    (fp_line (start -1.05 -1.5) (end -1.05 1.5)
+      (stroke (width 0.05) (type solid)) (layer "F.CrtYd"))
+    (fp_line (start -1.05 1.5) (end 8.67 1.5)
+      (stroke (width 0.05) (type solid)) (layer "F.CrtYd"))
+    (fp_line (start 8.67 -1.5) (end -1.05 -1.5)
+      (stroke (width 0.05) (type solid)) (layer "F.CrtYd"))
+    (fp_line (start 8.67 1.5) (end 8.67 -1.5)
+      (stroke (width 0.05) (type solid)) (layer "F.CrtYd"))
+    (fp_line (start 0 0) (end 0.66 0)
+      (stroke (width 0.1) (type solid)) (layer "F.Fab"))
+    (fp_line (start 0.66 -1.25) (end 0.66 1.25)
+      (stroke (width 0.1) (type solid)) (layer "F.Fab"))
+    (fp_line (start 0.66 1.25) (end 6.96 1.25)
+      (stroke (width 0.1) (type solid)) (layer "F.Fab"))
+    (fp_line (start 6.96 -1.25) (end 0.66 -1.25)
+      (stroke (width 0.1) (type solid)) (layer "F.Fab"))
+    (fp_line (start 6.96 1.25) (end 6.96 -1.25)
+      (stroke (width 0.1) (type solid)) (layer "F.Fab"))
+    (fp_line (start 7.62 0) (end 6.96 0)
+      (stroke (width 0.1) (type solid)) (layer "F.Fab"))
+    (pad "1" thru_hole circle (at 0 0 180) (size 1.6 1.6) (drill 0.8) (layers "*.Cu" "*.Mask")
+      (net 51 "Frontboard +3.3V") (pintype "passive"))
+    (pad "2" thru_hole oval (at 7.62 0 180) (size 1.6 1.6) (drill 0.8) (layers "*.Cu" "*.Mask")
+      (net 31 "Encoder left Frontboard") (pintype "passive"))
+    (model "${KICAD6_3DMODEL_DIR}/Resistor_THT.3dshapes/R_Axial_DIN0207_L6.3mm_D2.5mm_P7.62mm_Horizontal.wrl"
+      (offset (xyz 0 0 0))
+      (scale (xyz 1 1 1))
+      (rotate (xyz 0 0 0))
+    )
+  )
   (footprint "Capacitor_THT:C_Axial_L3.8mm_D2.6mm_P7.50mm_Horizontal" (layer "F.Cu")
     (at 86.1568 112.1318 90)
@@
   (segment (start 88.312099 47.95) (end 86.5632 49.698899) (width 0.25) (layer "B.Cu") (net 31))
   (segment (start 86.5632 89.11749) (end 96.29959 98.85388) (width 0.25) (layer "B.Cu") (net 31))
+  (segment (start 84.6836 74.2188) (end 86.5632 76.0984) (width 0.25) (layer "B.Cu") (net 31))
+  (segment (start 84.6836 72.8726) (end 84.6836 74.2188) (width 0.25) (layer "B.Cu") (net 31))
   (segment (start 96.29959 101.65388) (end 98.92688 101.65388) (width 0.25) (layer "B.Cu") (net 31))
   (segment (start 111.6588 49.125) (end 110.4838 47.95) (width 0.25) (layer "B.Cu") (net 31))
+  (segment (start 86.5632 49.698899) (end 86.5632 76.0984) (width 0.25) (layer "B.Cu") (net 31))
   (segment (start 110.4838 47.95) (end 88.312099 47.95) (width 0.25) (layer "B.Cu") (net 31))
   (segment (start 98.92688 101.65388) (end 101.9556 104.6826) (width 0.25) (layer "B.Cu") (net 31))
-  (segment (start 86.5632 49.698899) (end 86.5632 89.11749) (width 0.25) (layer "B.Cu") (net 31))
+  (segment (start 86.5632 76.0984) (end 86.5632 89.11749) (width 0.25) (layer "B.Cu") (net 31))
   (segment (start 96.29959 98.85388) (end 96.29959 101.65388) (width 0.25) (layer "B.Cu") (net 31))
   (segment (start 109.1188 49.125) (end 107.4938 47.5) (width 0.25) (layer "F.Cu") (net 32))
   (segment (start 87.1982 48.1838) (end 87.1982 89.75249) (width 0.25) (layer "F.Cu") (net 32))
+  (segment (start 85.1662 83.1342) (end 85.1662 87.72049) (width 0.25) (layer "F.Cu") (net 32))
+  (segment (start 85.1662 87.72049) (end 87.1982 89.75249) (width 0.25) (layer "F.Cu") (net 32))
   (segment (start 87.1982 89.75249) (end 91.29959 93.85388) (width 0.25) (layer "F.Cu") (net 32))
   (segment (start 107.4938 47.5) (end 87.882 47.5) (width 0.25) (layer "F.Cu") (net 32))
@@
   (segment (start 117.8306 129.832913) (end 117.8306 101.063056) (width 0.25) (layer "F.Cu") (net 51))
   (segment (start 108.756757 93.08688) (end 96.734 81.064123) (width 0.25) (layer "F.Cu") (net 51))
+  (segment (start 92.7862 80.3656) (end 95.2172 77.9346) (width 0.25) (layer "B.Cu") (net 51))
   (segment (start 96.734 59.0804) (end 95.2172 60.5972) (width 0.25) (layer "B.Cu") (net 51))
+  (segment (start 92.3036 75.021) (end 95.2172 77.9346) (width 0.25) (layer "B.Cu") (net 51))
+  (segment (start 92.7862 83.1342) (end 92.7862 80.3656) (width 0.25) (layer "B.Cu") (net 51))
   (segment (start 100.0252 59.055) (end 96.7594 59.055) (width 0.25) (layer "B.Cu") (net 51))
   (segment (start 95.2172 60.5972) (end 95.2172 77.9346) (width 0.25) (layer "B.Cu") (net 51))
@@
   (segment (start 100.0252 62.6872) (end 100.076 62.738) (width 0.25) (layer "B.Cu") (net 51))
   (segment (start 95.2172 77.9346) (end 91.29959 81.85221) (width 0.25) (layer "B.Cu") (net 51))
+  (segment (start 92.3036 72.8726) (end 92.3036 75.021) (width 0.25) (layer "B.Cu") (net 51))
   (segment (start 53.8226 76.5556) (end 57.5564 80.2894) (width 0.25) (layer "F.Cu") (net 52))
   (segment (start 53.8226 65.1064) (end 53.8226 76.5556) (width 0.25) (layer "F.Cu") (net 52))
