File: microlidian.kicad_sch (KiCad schematic)
At the start: 33 parts, among them J1 Eurorack power, J11 Backboard Conn 1, J12 Frontboard Conn 1, J13 Backboard Conn 2, J14 Frontboard Conn 2, J2 ST7789 TFT socket, J3 Expansion header, J4 ADS1015 digital side, J5 ADS1015 analog side, J7 TRS MIDI Out, SW1 RotaryEncoder_Switch, SW2 Back button, U1 SeeeduinoXIAO, U2 L78L05_TO92

Commit message: updated notes in readme and tracked most recent changes
Parts:
- added R5, R6: 10K, Resistor_THT:R_Axial_DIN0207_L6.3mm_D2.5mm_P7.62mm_Horizontal, symbol Device:R
Connections:
- net Encoder left Frontboard: now also R6.2
- net Encoder right Frontboard: now also R5.1
- net Frontboard +3.3V: now also R5.2, R6.1
Changed lines of the file:
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@@
   (junction (at 203.2 151.892) (diameter 0) (color 0 0 0 0)
   )
+  (junction (at 44.45 42.926) (diameter 0) (color 0 0 0 0)
+  )
   (junction (at 182.88 151.892) (diameter 0) (color 0 0 0 0)
   )
@@
   (junction (at 114.046 157.988) (diameter 0) (color 0 0 0 0)
   )
+  (junction (at 34.29 42.926) (diameter 0) (color 0 0 0 0)
+  )
   (wire (pts (xy 68.834 19.558) (xy 70.612 19.558))
     (stroke (width 0) (type default))
   )
+  (wire (pts (xy 22.733 42.926) (xy 34.29 42.926))
+    (stroke (width 0) (type default))
+  )
   (wire (pts (xy 182.88 151.892) (xy 190.5 151.892))
     (stroke (width 0) (type default))
@@
     (stroke (width 0) (type default))
   )
+  (wire (pts (xy 44.45 42.926) (xy 48.387 42.926))
+    (stroke (width 0) (type default))
+  )
   (wire (pts (xy 101.854 150.368) (xy 101.854 157.988))
     (stroke (width 0) (type default))
@@
     )
   )
+  (global_label "Frontboard +3.3V" (shape input) (at 15.113 42.926 90) (fields_autoplaced)
+    (effects (font (size 1.27 1.27)) (justify left))
+    (property "Intersheetrefs" "${INTERSHEET_REFS}" (at 15.113 23.7413 90)
+      (effects (font (size 1.27 1.27)) (justify left) hide)
+    )
+  )
+  (global_label "Frontboard +3.3V" (shape input) (at 56.007 42.926 90) (fields_autoplaced)
+    (effects (font (size 1.27 1.27)) (justify left))
+    (property "Intersheetrefs" "${INTERSHEET_REFS}" (at 56.007 23.7413 90)
+      (effects (font (size 1.27 1.27)) (justify left) hide)
+    )
+  )
   (global_label "Frontboard +5V" (shape input) (at 199.136 18.542 180) (fields_autoplaced)
     (effects (font (size 1.27 1.27)) (justify right))
@@
     )
   )
-  (global_label "Backboard GND" (shape input) (at 139.954 47.244 180) (fields_autoplaced)
-    (effects (font (size 1.27 1.27)) (justify right))
-    (property "Intersheetrefs" "${INTERSHEET_REFS}" (at 122.9464 47.244 0)
-      (effects (font (size 1.27 1.27)) (justify right) hide)
+  (global_label "Backboard GND" (shape input) (at 139.954 47.244 0) (fields_autoplaced)
+    (effects (font (size 1.27 1.27)) (justify left))
+    (property "Intersheetrefs" "${INTERSHEET_REFS}" (at 156.9616 47.244 0)
+      (effects (font (size 1.27 1.27)) (justify left) hide)
     )
   )
@@
     )
   )
+  (symbol (lib_id "Device:R") (at 18.923 42.926 90) (unit 1)
+    (in_bom yes) (on_board yes) (dnp no) (fields_autoplaced)
+    (property "Reference" "R6" (at 18.923 38.9001 90)
+      (effects (font (size 1.27 1.27)))
+    )
+    (property "Value" "10K" (at 18.923 40.8211 90)
+      (effects (font (size 1.27 1.27)))
+    )
+    (property "Footprint" "Resistor_THT:R_Axial_DIN0207_L6.3mm_D2.5mm_P7.62mm_Horizontal" (at 18.923 44.704 90)
+      (effects (font (size 1.27 1.27)) hide)
+    )
+    (property "Datasheet" "~" (at 18.923 42.926 0)
+      (effects (font (size 1.27 1.27)) hide)
+    )
+    (pin "1")
+    (pin "2")
+    (instances
+      (project "microlidian"
+        (path "/f3b5c3e2-a769-4f71-bc6f-5b90415c45e5"
+          (reference "R6") (unit 1)
+        )
+      )
+    )
+  )
   (symbol (lib_id "power:+12V") (at 182.88 146.812 90) (unit 1)
     (in_bom yes) (on_board yes) (dnp no) (fields_autoplaced)
@@
         )
       )
+    )
+  )
+  (symbol (lib_id "Device:R") (at 52.197 42.926 90) (unit 1)
+    (in_bom yes) (on_board yes) (dnp no) (fields_autoplaced)
+    (property "Reference" "R5" (at 52.197 38.9001 90)
+      (effects (font (size 1.27 1.27)))
+    )
+    (property "Value" "10K" (at 52.197 40.8211 90)
+      (effects (font (size 1.27 1.27)))
+    )
+    (property "Footprint" "Resistor_THT:R_Axial_DIN0207_L6.3mm_D2.5mm_P7.62mm_Horizontal" (at 52.197 44.704 90)
+      (effects (font (size 1.27 1.27)) hide)
+    )
+    (property "Datasheet" "~" (at 52.197 42.926 0)
+      (effects (font (size 1.27 1.27)) hide)
+    )
+    (pin "1")
+    (pin "2")
+    (instances
+      (project "microlidian"
+        (path "/f3b5c3e2-a769-4f71-bc6f-5b90415c45e5"
+          (reference "R5") (unit 1)
+        )
+      )
